File: PCB/Impedance-measurement-3/Project-1-backups/Project-1_before_user_edit_fixes_20260705_204359.kicad_pcb (KiCad board)
At the start: 2 copper layers, 171 x 114 mm, 73 parts, among them U1 STM32F303CCT6

Commit message: mounting holes included 6/7/2026
Parts:
- removed REF** (x4): MountingHole_3.2mm_M3_Pad, MountingHole:MountingHole_3.2mm_M3_Pad
Connections:
- Precision-OP-Amp1 pad 5: GND -> (no net)
- Precision-OP-Amp1 pad 6: unused_Precision-OP-Amp1_ChB_buffer -> (no net)
- Precision-OP-Amp1 pad 7: unused_Precision-OP-Amp1_ChB_buffer -> (no net)
- Precision-OP-Amp2 pad 5: GND -> (no net)
- Precision-OP-Amp2 pad 6: unused_Precision-OP-Amp2_ChB_buffer -> (no net)
- Precision-OP-Amp2 pad 7: unused_Precision-OP-Amp2_ChB_buffer -> (no net)
Routing:
- net (no net): track 0.00 -> 2.54 mm
- net unused_Precision-OP-Amp1_ChB_buffer: track 1.27 -> 0.00 mm
- net unused_Precision-OP-Amp2_ChB_buffer: track 1.27 -> 0.00 mm
