File: PCB/Impedance-measurement-3/Project-1-backups/Project-1-2026-07-24_185750/Project-1.kicad_pcb (KiCad board)
At the start: 2 copper layers, 112 x 88 mm, 74 parts, among them J2 USB_C_Receptacle, U1 STM32F303CCT6, U2 W25Q32JVSSIQ, U5 LM7805_TO220, U9 OPA4141AID

Commit message: schematic and layout changed 25/7/2026
Routing:
- net Net-(USB-UART(CP2102)1-NC-Pad10): track 10.0 -> 23.6 mm
- net Net-(U9-V-): track 7.89 -> 0.00 mm
- net GND: track 652.4 -> 650.7 mm
Changed lines of the file:
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@@
 		(tags "capacitor")
 		(property "Reference" "C8-100nF1"
-			(at 0 -1.68 0)
+			(at 0 -1.68 360)
 			(layer "F.SilkS")
 			(effects
@@
 		)
 		(property "Value" "100nF"
-			(at 0 1.68 0)
+			(at 0 1.68 360)
 			(layer "F.Fab")
 			(effects
@@
 		)
 		(fp_text user "${REFERENCE}"
-			(at 0 0 0)
+			(at 0 0 360)
 			(layer "F.Fab")
 			(effects
@@
 	)
 	(segment
-		(start 78.5 80.55)
-		(end 82.95 85)
-		(width 0.1)
-		(layer "F.Cu")
-		(net 4)
-	)
-	(segment
 		(start 121.05 46)
 		(end 114.07 46)
@@
 	)
 	(segment
+		(start 74.475 80.55)
+		(end 74.475 81.82)
+		(width 0.1)
+		(layer "F.Cu")
+		(net 4)
+	)
+	(segment
 		(start 67.165 50.32)
 		(end 66.2 50.32)
@@
 	)
 	(segment
+		(start 80.05 84)
+		(end 81.05 85)
+		(width 0.1)
+		(layer "F.Cu")
+		(net 4)
+	)
+	(segment
 		(start 127.25 103.25)
 		(end 131 107)
@@
 	)
 	(segment
+		(start 78.91 84)
+		(end 78 83.09)
+		(width 0.1)
+		(layer "F.Cu")
+		(net 4)
+	)
+	(segment
 		(start 94 58)
 		(end 94 59)
@@
 	)
 	(segment
-		(start 74.475 80.55)
-		(end 78.5 80.55)
-		(width 0.1)
-		(layer "F.Cu")
-		(net 4)
-	)
-	(segment
 		(start 89.05 82)
 		(end 90.05 81)
@@
 	)
 	(segment
+		(start 74.475 83.09)
+		(end 78 83.09)
+		(width 0.1)
+		(layer "F.Cu")
+		(net 4)
+	)
+	(segment
 		(start 72 81)
 		(end 72.45 80.55)
@@
 	)
 	(segment
+		(start 78.91 84)
+		(end 80.05 84)
+		(width 0.1)
+		(layer "F.Cu")
+		(net 4)
+	)
+	(segment
 		(start 135 75)
 		(end 136 75)
@@
 	)
 	(segment
-		(start 142.63 52.32)
-		(end 142.63 52.82)
+		(start 142.63 51.82)
+		(end 142.63 51.32)
 		(width 0.1)
 		(layer "F.Cu")
@@
 	)
 	(segment
-		(start 145.5 49.965001)
-		(end 144.534999 49)
+		(start 140.32 52.32)
+		(end 140 52)
 		(width 0.1)
 		(layer "F.Cu")
@@
 	)
 	(segment
-		(start 142.63 54.32)
-		(end 143.5 55.19)
+		(start 141.82 53.82)
+		(end 141 53)
 		(width 0.1)
 		(layer "F.Cu")
@@
 	)
 	(segment
-		(start 145.5 50.45)
-		(end 145.5 49.965001)
+		(start 140 52)
+		(end 140.68 51.32)
 		(width 0.1)
 		(layer "F.Cu")
@@
 	)
 	(segment
-		(start 142.63 53.32)
-		(end 142.63 53.82)
+		(start 142.63 51.32)
+		(end 143.5 50.45)
 		(width 0.1)
 		(layer "F.Cu")
@@
 	)
 	(segment
-		(start 142.63 51.82)
-		(end 142.63 52.32)
+		(start 143.5 55.19)
+		(end 142.63 54.32)
+		(width 0.1)
+		(layer "F.Cu")
+		(net 64)
+	)
+	(segment
+		(start 142.63 52.32)
+		(end 140.32 52.32)
+		(width 0.1)
+		(layer "F.Cu")
+		(net 64)
+	)
+	(segment
+		(start 140.68 51.32)
+		(end 142.63 51.32)
+		(width 0.1)
+		(layer "F.Cu")
+		(net 64)
+	)
+	(segment
+		(start 145.5 49.965001)
+		(end 144.534999 49)
+		(width 0.1)
+		(layer "F.Cu")
+		(net 64)
+	)
+	(segment
+		(start 142.63 53.32)
+		(end 141.32 53.32)
 		(width 0.1)
 		(layer "F.Cu")
@@
 	)
 	(segment
-		(start 142.63 52.82)
-		(end 142.63 53.32)
+		(start 141.32 53.32)
+		(end 141 53)
 		(width 0.1)
 		(layer "F.Cu")
@@
 	)
 	(segment
-		(start 144.534999 49)
-		(end 144 49)
+		(start 145.5 50.45)
+		(end 145.5 49.965001)
 		(width 0.1)
 		(layer "F.Cu")
@@
 	)
 	(segment
-		(start 143.5 50.45)
-		(end 142.63 51.32)
+		(start 142.63 52.82)
+		(end 142.63 52.32)
 		(width 0.1)
 		(layer "F.Cu")
@@
 	)
 	(segment
-		(start 142.63 51.32)
-		(end 142.63 51.82)
+		(start 140.32 54.32)
+		(end 140 54)
+		(width 0.1)
+		(layer "F.Cu")
+		(net 64)
+	)
+	(segment
+		(start 140 54)
+		(end 140 52)
 		(width 0.1)
 		(layer "F.Cu")
@@
 	(segment
 		(start 142.63 53.82)
-		(end 142.63 54.32)
+		(end 141.82 53.82)
 		(width 0.1)
 		(layer "F.Cu")
@@
 	)
 	(segment
-		(start 144 50.45)
-		(end 143.5 50.45)
+		(start 143.5 50.45)
+		(end 144 50.45)
 		(width 0.1)
 		(layer "F.Cu")
@@
 	)
 	(segment
-		(start 74.475 85.63)
-		(end 74.475 84.36)
+		(start 144.534999 49)
+		(end 144 49)
 		(width 0.1)
 		(layer "F.Cu")
-		(net 81)
+		(net 64)
 	)
 	(segment
-		(start 81.05 85)
-		(end 77.87 81.82)
+		(start 142.63 54.32)
+		(end 140.32 54.32)
 		(width 0.1)
 		(layer "F.Cu")
-		(net 82)
+		(net 64)
 	)
 	(segment
-		(start 77.87 81.82)
-		(end 74.475 81.82)
+		(start 141 53)
+		(end 140 52)
+		(width 0.1)
+		(layer "F.Cu")
+		(net 64)
+	)
+	(segment
+		(start 74.475 85.63)
+		(end 74.475 84.36)
 		(width 0.1)
 		(layer "F.Cu")
-		(net 82)
+		(net 81)
 	)
 	(zone
