File: PCB/Impedance-measurement-3/Project-1-backups/Project-1-2026-07-24_185750/Project-1-backups/Project-1_before_100nF_caps_20260719_213557.kicad_pcb (KiCad board)
At the start: 2 copper layers, 112 x 88 mm, 74 parts, among them J2 USB_C_Receptacle, U1 STM32F303CCT6, U2 W25Q32JVSSIQ, U5 LM7805_TO220, U9 OPA4141AID

Commit message: schematic and layout changed 25/7/2026
Parts:
- moved C18-100nF1 119.1 mm to (37.1, 45.0)
- moved C5-100nF1 116.2 mm to (46.0, 45.0), turned to 0 degrees
- moved C28-100nF1 114.5 mm to (41.6, 45.0)
- moved C19-100nF1 100.9 mm to (37.1, 48.0)
- moved C4-100nF1 94.4 mm to (41.6, 54.0)
- moved C17-100nF2 92.9 mm to (32.7, 54.0)
- moved C3-100nF1 88.2 mm to (41.6, 48.0)
- moved C9-100nF1 76.4 mm to (46.0, 54.0)
- moved C8-100nF1 75.0 mm to (46.0, 51.0), turned to 0 degrees
- moved C17-100nF1 72.5 mm to (32.7, 51.0), turned to 0 degrees
- moved C6-100nF1 55.8 mm to (46.0, 48.0)
- moved C2-100nF1 54.3 mm to (37.1, 51.0), turned to 0 degrees
- moved C16-100nF1 53.5 mm to (32.7, 48.0), turned to 0 degrees
- moved C3-100nF2 52.8 mm to (41.6, 51.0)
- moved C15-100nF1 52.5 mm to (32.7, 45.0), turned to 0 degrees
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Connections:
- C3-100nF2 pad 1: Net-(U9-V-) -> GND
- U9 pad 11: Net-(U9-V-) -> GND
Routing:
- net GND: track 652.4 -> 578.1 mm, vias 41 -> 36
- net VDD: track 316.0 -> 269.2 mm, vias 24 -> 13
- net /VBUS-5V: track 347.9 -> 320.4 mm, vias 14 -> 11
- net Net-(USB-UART(CP2102)1-NC-Pad10): track 10.0 -> 23.6 mm
- net /M-NRST: track 125.6 -> 116.6 mm, vias 8 -> 5
- net Net-(U9-V-): track 7.89 -> 0.00 mm
- net Net-(USB-UART(CP2102)1-DTR): track 19.3 -> 24.8 mm, vias 2 -> 3
- net /M-VREF+: track 85.6 -> 82.8 mm
- net Net-(Signal-generator2-CAP/2.5V): track 10.2 -> 8.98 mm
- net Net-(SWD-connector1-SWDCLK): track 275.5 -> 276.1 mm
