File: PCB/Impedance-measurement-3/Project-1-backups/Project-1-2026-07-24_185750/Project-1-backups/Project-1_before_clearance_fix_20260717_195956.kicad_pcb (KiCad board)
At the start: 2 copper layers, 112 x 88 mm, 74 parts, among them J2 USB_C_Receptacle, U1 STM32F303CCT6, U2 W25Q32JVSSIQ, U5 LM7805_TO220, U9 OPA4141AID

Commit message: schematic and layout changed 25/7/2026
Parts:
- removed C16-100nF1, C17-100nF2, C18-100nF1, C19-100nF1, C28-100nF1: 100nF, Capacitor_SMD:C_0805_2012Metric
- added REF**: MountingHole_3.2mm_M3_Pad, MountingHole:MountingHole_3.2mm_M3_Pad, F.Cu at (164.0, 112.0)
- added REF**: MountingHole_3.2mm_M3_Pad, MountingHole:MountingHole_3.2mm_M3_Pad, F.Cu at (64.0, 112.0)
- added REF**: MountingHole_3.2mm_M3_Pad, MountingHole:MountingHole_3.2mm_M3_Pad, F.Cu at (64.0, 36.0)
- added REF**: MountingHole_3.2mm_M3_Pad, MountingHole:MountingHole_3.2mm_M3_Pad, F.Cu at (164.0, 36.0)
- C15-100nF1, C17-100nF1, C2-100nF1, C21-100nF1, C3-100nF1, C3-100nF2, C4-100nF1, C5-100nF1, C6-100nF1, C8-100nF1, C9-100nF1: footprint Capacitor_SMD:C_0805_2012Metric -> Capacitor_THT:C_Axial_L3.8mm_D2.6mm_P7.50mm_Horizontal
- moved C8-100nF1 14.1 mm to (116.0, 99.6), turned to 90 degrees
- moved C17-100nF1 12.1 mm to (88.2, 80.8), turned to 0 degrees
- moved C6-100nF1 10.1 mm to (101.0, 79.6), turned to 90 degrees
- moved C15-100nF1 9.62 mm to (84.0, 65.6), turned to 90 degrees
- moved C9-100nF1 7.39 mm to (121.0, 53.3), turned to 90 degrees
- moved C3-100nF2 6.80 mm to (84.0, 91.5), turned to 90 degrees
- moved C2-100nF1 5.87 mm to (77.2, 78.8), turned to 0 degrees
- moved C3-100nF1 5.47 mm to (129.6, 54.6), turned to -90 degrees
- moved C5-100nF1 4.80 mm to (155.0, 72.2), turned to -90 degrees
- moved C21-100nF1 3.19 mm to (84.0, 46.1), turned to -90 degrees
- moved C4-100nF1 1.79 mm to (136.6, 54.3), turned to -90 degrees
Connections:
- C17-100nF1 pad 1: VDD -> GND
- C17-100nF1 pad 2: GND -> VDD
- C2-100nF1 pad 1: GND -> /VBUS-5V
- C2-100nF1 pad 2: /VBUS-5V -> GND
- C21-100nF1 pad 1: GND -> /VBUS-5V
- C21-100nF1 pad 2: /VBUS-5V -> GND
- C3-100nF1 pad 1: /M-NRST -> Net-(USB-UART(CP2102)1-DTR)
- C3-100nF1 pad 2: Net-(USB-UART(CP2102)1-DTR) -> /M-NRST
- C3-100nF2 pad 1: Net-(U9-V-) -> GND
- C4-100nF1 pad 1: GND -> VDD
- C4-100nF1 pad 2: VDD -> GND
- C5-100nF1 pad 1: GND -> /M-NRST
- C5-100nF1 pad 2: /M-NRST -> GND
- C6-100nF1 pad 1: GND -> VDD
- C6-100nF1 pad 2: VDD -> GND
- C8-100nF1 pad 1: GND -> VDD
- C8-100nF1 pad 2: VDD -> GND
- C9-100nF1 pad 1: GND -> VDD
- C9-100nF1 pad 2: VDD -> GND
- U9 pad 11: Net-(U9-V-) -> GND
Routing:
- net GND: track 652.4 -> 578.1 mm, vias 41 -> 36
- net VDD: track 316.0 -> 269.2 mm, vias 24 -> 13
- net /VBUS-5V: track 347.9 -> 320.4 mm, vias 14 -> 11
- net Net-(USB-UART(CP2102)1-NC-Pad10): track 10.0 -> 23.6 mm
- net /M-NRST: track 125.6 -> 116.6 mm, vias 8 -> 5
- net Net-(U9-V-): track 7.89 -> 0.00 mm
- net Net-(USB-UART(CP2102)1-DTR): track 19.3 -> 24.8 mm, vias 2 -> 3
- net /M-VREF+: track 85.6 -> 82.8 mm
- net Net-(U1-PA1): track 158.1 -> 160.2 mm, vias 3 -> 4
- net /Electrode1: track 106.4 -> 105.1 mm
- net Net-(Signal-generator2-CAP/2.5V): track 10.2 -> 8.98 mm
- net Net-(U9-+IN_B): track 128.7 -> 129.4 mm
- net Net-(Signal-generator2-SCLK): track 57.8 -> 58.5 mm
- net Net-(SWD-connector1-SWDCLK): track 275.5 -> 276.1 mm
